File: 8701Duo.kicad_pcb (KiCad board)
At the start: 2 copper layers, 19.5 x 21 mm, 12 parts, among them J1 Clock, U1 ICS525-01R, U2 MOS8701, U3 74LVC1G06, X1 LFSPXO021772Bulk, X2 LFSPXO020648Bulk

Commit message: Add files via upload
Connections:
- J1 pad 2: Net-(J1-Pad2) -> Net-(J1-Pad1)
- U1 pad 4: Net-(J1-Pad2) -> Net-(J1-Pad1)
- U3 pad 2: Net-(J1-Pad2) -> Net-(J1-Pad1)
- X1 pad 1: Net-(J1-Pad2) -> Net-(J1-Pad1)
Routing:
- net Net-(J1-Pad1): track 6.04 -> 46.3 mm, vias 0 -> 2
- net Net-(J1-Pad2): track 39.4 -> 0.00 mm, vias 2 -> 0

Commit message: Add files via upload
Parts:
- removed X1: LFSPXO021772Bulk, Oscillator:Oscillator_SMD_IQD_IQXO70-4Pin_7.5x5.0mm
- added 14.3MHz: LFSPXO021772Bulk, Oscillator:Oscillator_SMD_IQD_IQXO70-4Pin_7.5x5.0mm, F.Cu at (93.9, 66.2)
- moved 17.7MHz 8.13 mm to (93.9, 74.3)
- renumbered X2 to 17.7MHz
Other:
- board text added: "N P"
- board text removed: "P N"
Changed lines of the file:
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@@
   (page A4)
   (layers
-    (0 F.Cu signal)
-    (31 B.Cu signal)
+    (0 F.Cu signal hide)
+    (31 B.Cu signal hide)
     (32 B.Adhes user hide)
     (33 F.Adhes user hide)
@@
   )
   (setup
-    (last_trace_width 0.539)
+    (last_trace_width 0.25)
     (user_trace_width 0.275)
     (user_trace_width 0.35)
@@
   )
   (module Oscillator:Oscillator_SMD_IQD_IQXO70-4Pin_7.5x5.0mm (layer F.Cu)
-    (at 93.9165 74.295 90)
+    (at 93.9165 66.167 90)
     (descr "IQD Crystal Clock Oscillator IQXO-70, http://www.iqdfrequencyproducts.com/products/details/iqxo-70-11-30.pdf, 7.5x5.0mm^2 package")
     (tags "SMD SMT crystal oscillator")
     (attr smd)
-    (fp_text reference X1 (at 0 -4.1 90) (layer F.SilkS)
+    (fp_text reference 14.3MHz (at 0 0 90) (layer F.SilkS)
       (effects (font (size 1 1) (thickness 0.15)))
     )
@@
   )
   (module Oscillator:Oscillator_SMD_IQD_IQXO70-4Pin_7.5x5.0mm (layer F.Cu)
-    (at 93.9165 66.167 90)
+    (at 93.9165 74.295 90)
     (descr "IQD Crystal Clock Oscillator IQXO-70, http://www.iqdfrequencyproducts.com/products/details/iqxo-70-11-30.pdf, 7.5x5.0mm^2 package")
     (tags "SMD SMT crystal oscillator")
     (attr smd)
-    (fp_text reference X2 (at 0 -4.1 90) (layer F.SilkS)
+    (fp_text reference 17.7MHz (at 0 0 90) (layer F.SilkS)
       (effects (font (size 1 1) (thickness 0.15)))
     )
@@
   (target plus (at 88.9 76.2) (size 5) (width 0.05) (layer Edge.Cuts))
   (target plus (at 88.9 63.5) (size 5) (width 0.05) (layer Edge.Cuts))
-  (gr_text "P  N" (at 93.9165 62.992) (layer B.SilkS)
+  (gr_text "N  P" (at 93.9165 62.992) (layer B.SilkS)
     (effects (font (size 2 2) (thickness 0.3)) (justify mirror))
   )
